File: HARDWARE/ETH1ISO224/ETH1ISO224.kicad_sch (KiCad schematic)
At the start: 0 parts

Commit message: Hardware design
Parts:
- added FID101, FID102, FID103, FID104: Fiducial, Fiducial:Fiducial_1.5mm_Mask3mm, symbol Mechanical:Fiducial
- added H101, H102: M3, MountingHole:MountingHole_3.2mm_M3_DIN965, symbol Mechanical:MountingHole
- added H103, H104: M3, MountingHole:MountingHole_3.2mm_M3_DIN965_Pad, symbol Mechanical:MountingHole
- added HS101: 960-19-12-S-AB-0, ETH1ISO224:960-19-12-S-AB-0, symbol Mechanical:Heatsink
Other:
- note added: "TG-A2200-10-10-1.5"

Commit message: Hardware design done
Parts:
- FID101, FID102, FID103, FID104: now left out of the parts list
Changed lines of the file:
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@@
 		(unit 1)
 		(exclude_from_sim no)
-		(in_bom yes)
+		(in_bom no)
 		(on_board yes)
 		(dnp no)
@@
 		(unit 1)
 		(exclude_from_sim no)
-		(in_bom yes)
+		(in_bom no)
 		(on_board yes)
 		(dnp no)
@@
 		(unit 1)
 		(exclude_from_sim no)
-		(in_bom yes)
+		(in_bom no)
 		(on_board yes)
 		(dnp no)
@@
 		(unit 1)
 		(exclude_from_sim no)
-		(in_bom yes)
-		(on_board yes)
-		(dnp no)
+		(in_bom no)
+		(on_board yes)
+		(dnp no)
