File: HARDWARE/ETH1ISO224/Analog.kicad_sch (KiCad schematic)
At the start: 53 parts, among them J201 1710072, U201 ISO224, U202 TBA1-0513E, U203 DG419LEDY, U204 DG412LEDQ, U205 OPA2340UA, U206 REF1925AIDDCT

Commit message: Hardware design
Parts:
- removed L201: MGDQ4-00004-P, symbol Device:L
- added R220, R223: 0, Resistor_SMD:R_0603_1608Metric_Pad0.98x0.95mm_HandSolder, symbol Device:R
- added R221, R225: 100k/.05%, Resistor_SMD:R_0603_1608Metric_Pad0.98x0.95mm_HandSolder, symbol Device:R
- added R224: 3k/.05%, Resistor_SMD:R_0603_1608Metric_Pad0.98x0.95mm_HandSolder, symbol Device:R
- added RN201: 1776-C68xx, ETH1ISO224:1776-C68xx, symbol ETH1ISO224:1776-C68xx
- C201: value 10n/1k-2k -> 10n/2k
- C205: footprint ETH1ISO224:NX5032GA -> Capacitor_SMD:C_0603_1608Metric_Pad1.08x0.95mm_HandSolder
- E201: value SparkGap -> 2087-150-SM-RPLF; footprint (none) -> ETH1ISO224:2087
- R210, R211, R212, R213: value 10k/0.1% -> 10k/.05%
- R216: value 180k/0.05% -> 180k/.05%
- R217: value 18k/0.05% -> 18k/.05%
- R218: value 2k/0.05% -> 2k/.05%
- RV201: value B72660M0301 -> B72650M0301; footprint (none) -> Varistor:Varistor_Panasonic_VF
- renumbered R206 to R204, R204 to R205, R205 to R206, R220 to R222, R221 to R226, RN201 to RN202, RN202 to RN203, RN203 to RN204
Connections:
- net +1V25: now also R223.1
- net +2V5: now also C210.2, R212.1, RN202.2, R221.1
- net GND: now also R225.1; no longer C210.2, R212.1, RN202.2
- net GND1: now also RN201.6 (R5)
- net VOUT: now also R220.2; no longer R219.2
- net at R201.2: now also E201.2, J201.1 (Pin_1), RN201.1 (common)
- net at R208.1, R209.2, U201.2 (IN): now also RN201.3 (R2)
- new net: R219.2, R220.1
- new net: R221.2, R224.1
- new net VCOM: R223.2, R224.2, R225.2
- no-connect marks 0 -> 3
Other:
- note added: "Common voltage selection."
- moved on the sheet: C201, C202, C203, C204, C205, C206, C207, C208, C209, C210, C213, C214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

Commit message: Hardware design
Parts:
- added L201: 74438335100, Inductor_SMD:L_Wuerth_MAPI-3015, symbol Device:L
- renumbered R205 to R204, R206 to R205, R204 to R206, R222 to R220, R226 to R221, R223 to R222, R221 to R223, R225 to R224, R224 to R225, R220 to R226, RN202 to RN201, RN203 to RN202, RN204 to RN203, RN201 to RN204
Connections:
- net at R201.2, RN204.1 (common): now also L201.2; no longer E201.2, J201.1 (Pin_1)
- new net: E201.2, J201.1 (Pin_1), L201.1
Other:
- moved on the sheet: C201, E201, J201, R204, R205, RV201

Commit message: Hardware design
Parts:
- added C219, C220, C221, C222, C223: 0.1u, Capacitor_SMD:C_0603_1608Metric_Pad1.08x0.95mm_HandSolder, symbol Device:C
- R219: value 100k/0.05% -> 51k/.05%
- R223: value 100k/.05% -> 51k/.05%
- R225: value 3k/.05% -> 511/.05%
- R226: value 0 -> 511/.05%
Connections:
- net +3.3V: now also C222.1, C223.1
- net +5V: no longer C206.1, C207.1, C208.1, U202.1 (+Vin)
- net +5VA: now also C206.1, C207.1, C208.1, U202.1 (+Vin), C219.1, C220.1, C221.1
- net GND: now also C219.2, C220.2, C221.2, C222.2, C223.2
Other:
- moved on the sheet: C201, C202, C203, C204, C206, C207, C208, R204, R205, R209, R222, R223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

Commit message: Hardware design
Parts:
- added SYM201, SYM202: SYM_Flash_Small, ETH1ISO224:Symbol_Attention_Triangle_8x7mm_Copper, symbol Graphic:SYM_Flash_Small
- U202: value TBA1-0513E -> TBA 1-0511HI; footprint Converter_DCDC:Converter_DCDC_TRACO_TBA1-xxxxE_Single_THT -> ETH1ISO224:TBA1
Other:
- moved on the sheet: C213, C214, U206

Commit message: Hardware design
Parts:
- removed C213, C216, C218: 1u, Capacitor_SMD:C_0603_1608Metric_Pad1.08x0.95mm_HandSolder, symbol Device:C
- removed C214, C215, C217: 0.1u, Capacitor_SMD:C_0603_1608Metric_Pad1.08x0.95mm_HandSolder, symbol Device:C
- removed R219, R223: 51k/.05%, Resistor_SMD:R_0603_1608Metric_Pad0.98x0.95mm_HandSolder, symbol Device:R
- removed R222: 0, Resistor_SMD:R_0603_1608Metric_Pad0.98x0.95mm_HandSolder, symbol Device:R
- removed R224: 100k/.05%, Resistor_SMD:R_0603_1608Metric_Pad0.98x0.95mm_HandSolder, symbol Device:R
- removed R225, R226: 511/.05%, Resistor_SMD:R_0603_1608Metric_Pad0.98x0.95mm_HandSolder, symbol Device:R
- removed RN203: MPMT2003AT5, Package_TO_SOT_SMD:SOT-23, symbol Device:VoltageDivider_CenterPin3
- removed U206: REF1925AIDDCT, Package_TO_SOT_SMD:SOT-23-5_HandSoldering, symbol ETH1ISO224:REF19xxAIDDCT
- added C211: 0.1u, Capacitor_SMD:C_0603_1608Metric_Pad1.08x0.95mm_HandSolder, symbol Device:C
- added D201: 1N4148W, Diode_SMD:D_SOD-123, symbol Diode:1N4148W
- added U206: LT6015IS5, Package_TO_SOT_SMD:SOT-23-5, symbol Amplifier_Operational:LT6015xS5
- R210: renamed from R221; value 100k -> 10k
- R213: renamed from R212; value 10k/.05% -> 5k/.05%
- R214: renamed from R213; value 10k/.05% -> 5k/.05%
- R216: renamed from R215; value 100k/0.1% -> 100k/0.05%
- R220: value 100k/0.05% -> 0
- RN202: renamed from RN201; value MPMT2003AT5 -> MPMT50011002AT5
- RN203: renamed from RN202; value MPMT2003AT5 -> MPMT50011002AT5
- U203: renamed from U202; footprint ETH1ISO224:TBA1 -> ETH1ISO224:TBA 1HI; symbol Converter_DCDC:TBA1-0513E -> ETH1ISO224:TBA 1-0511HI
- renumbered C221 to C212, C219 to C213, C220 to C214, C222 to C215, C223 to C216, C211 to C217, C212 to C218, R210 to R211, R211 to R212, R214 to R215, R216 to R217, R217 to R218, R218 to R219, RN204 to RN201, U204 to U201, U201 to U202, U203 to U204
Connections:
- net +15V: now also U203.7 (+Vout); no longer U203.6 (+Vout)
- net +3.3V: now also U206.3 (+)
- net +5VA: now also C211.1, U206.5 (V+)
- net GND: now also C211.2, U206.2 (V-); no longer R220.1
- net GND1: now also U203.5 (-Vout); no longer U203.4 (-Vout)
- net VCOM: now also C210.2, R213.1, R215.2, R216.2, R219.2, RN202.1
- net at R211.1, U202.7 (OUT+): now also RN202.2; no longer RN202.1
- net at R217.1, U201.3, U205.7: now also R220.1, D201.2 (A), U206.4 (-)
- net at C209.2, R214.2, U204.2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: now also RN203.1; no longer RN203.2
- net at R212.1, U202.6 (OUT-): now also RN203.2; no longer RN203.1
- removed net +2V5: C210.2, R213.1, R215.2, R216.2, R219.2, RN202.2
- new net: D201.1 (K), U206.1
Other:
- note added: "Voltage clipper"
- note removed: "Common voltage selection."
- moved on the sheet: C201, C202, C203, C204, C205, C206, C207, C208, C209, C210, C212, C213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

Commit message: Hardware design done
Parts:
- removed R201: 6k19, Resistor_SMD:R_1206_3216Metric_Pad1.30x1.75mm_HandSolder, symbol Device:R
- added C211: 0.1u, Capacitor_SMD:C_0603_1608Metric_Pad1.08x0.95mm_HandSolder, symbol Device:C
- added R214: 0, Resistor_SMD:R_0603_1608Metric_Pad0.98x0.95mm_HandSolder, symbol Device:R
- added R221: 1k, Resistor_SMD:R_0603_1608Metric_Pad0.98x0.95mm_HandSolder, symbol Device:R
- added U208: MCP6001-OT, Package_TO_SOT_SMD:SOT-23-5, symbol Amplifier_Operational:MCP6001-OT
- C201: value 10n/2k -> 0.01u/1.5k
- L201: value 74438335100 -> 74438336100
- U202: renamed from U203; value TBA 1-0511HI -> TBA 1-0513HI
- renumbered C211 to C212, C212 to C213, C213 to C214, C214 to C215, C215 to C216, C216 to C217, C217 to C218, C218 to C219, R202 to R201, R203 to R202, R206 to R203, R207 to R206, R208 to R207, R209 to R208, R211 to R209, R212 to R210, R213 to R211, R214 to R212, R215 to R213, R216 to R215, R217 to R216, R218 to R217, R219 to R218, R220 to R219, R210 to R220, U202 to U201, U204 to U203, U201 to U204, U206 to U207
Connections:
- net +5VA: now also C211.1, U208.5 (V+)
- net GND: now also C211.2, U208.2 (V-)
- net VCOM: now also R214.1, U208.3 (+); no longer R215.2, R218.2
- net at R201.2: now also L201.2, RN201.1 (common)
- net at R216.1, U204.3, U205.7: now also R221.1; no longer D201.2 (A), R219.1, U207.4 (-)
- new net: R214.2, R215.2, R218.2, U208.1, U208.4 (-)
- new net: D201.2 (A), R219.1, R221.2, U207.4 (-)
Other:
- note added: "NOTE: LT6015 can't be replaced with diff. op amp."
- moved on the sheet: C201, C202, C203, C204, C205, C206, C207, C208, C209, C210, C212, C213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

Commit message: Software development
Parts:
- R213: value 0 -> 10k
Other:
- note added: "Delete this"
Changed lines of the file:
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@@
 		)
 	)
+	(text "Delete this"
+		(exclude_from_sim no)
+		(at 267.716 66.04 0)
+		(effects
+			(font
+				(size 1.27 1.27)
+			)
+		)
+	)
 	(text "NOTE: LT6015 can't be replaced with diff. op amp."
 		(exclude_from_sim no)
@@
 			)
 		)
-		(property "Value" "0"
+		(property "Value" "10k"
 			(at 160.655 71.12 0)
 			(effects
