File: HARDWARE/ETH1ISO224/ETH1ISO224.kicad_pcb (KiCad board)
At the start: 4 copper layers, 100 x 45 mm, 147 parts, among them J201 1710072, J301 1715721, J401 20021111-00010T4LF, J501 RJ45_Wuerth_7499010121A, Q301 SI5618A, Q302 MMBT3904, U201 ISO224, U202 TBA 1-0513HI, U203 DG419LEDY, U204 DG412LEDQ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

Commit message: Software development
Parts:
- R213: value 0 -> 10k
- U402: value REF1933AIDDCT -> REF2033AIDDCT
Routing:
- net Net-(R204-Pad2): track 1.52 -> 3.73 mm
- net GND1: track 98.3 -> 99.9 mm

Commit message: PCB changes
Parts:
- moved SYM201 28.8 mm to (111.3, 101.7)
Changed lines of the file:
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@@
 	(footprint "ETH1ISO224:Symbol_Attention_Triangle_8x7mm_Copper"
 		(layer "F.Cu")
-		(at 108.077 73.152)
+		(at 111.252 101.727)
 		(descr "Symbol, Attention, 8x7mm, copper layer")
 		(tags "warning graphic")
@@
 	)
 	(gr_line
+		(start 103.632 101.346)
+		(end 103.632 98.552)
+		(stroke
+			(width 0.5)
+			(type default)
+		)
+		(layer "F.SilkS")
+	)
+	(gr_line
 		(start 141.5415 104.4575)
 		(end 141.5415 105.0925)
@@
 	)
 	(gr_line
+		(start 103.632 76.2)
+		(end 103.632 73.406)
+		(stroke
+			(width 0.5)
+			(type default)
+		)
+		(layer "F.SilkS")
+	)
+	(gr_line
 		(start 164.2745 93.2815)
 		(end 164.9095 93.2815)
@@
 			(type default)
 		)
+		(layer "F.SilkS")
+	)
+	(gr_line
+		(start 102.235 74.803)
+		(end 105.029 74.803)
+		(stroke
+			(width 0.5)
+			(type default)
+		)

Commit message: PCB changes
Other:
- outline, holes or cut-outs redrawn
- board text added: "ETH1ISO224 V1.2 Default IP : 192.168.1.21"
- board text removed: "ETH1ISO224 V1.1 Default IP : 192.168.1.21"
Changed lines of the file:
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@@
 		(at 126.238 105.664 180)
 		(property "Reference" "U202"
-			(at 1.016 3.937 0)
+			(at 2.413 3.937 0)
 			(unlocked yes)
 			(layer "F.SilkS")
@@
 	)
 	(gr_line
-		(start 128.778 66.167)
-		(end 128.778 109.093)
+		(start 127.5 66)
+		(end 127.5 98.5)
 		(stroke
 			(width 0.3)
@@
 	)
 	(gr_line
-		(start 128.778 66.167)
-		(end 128.778 89.916)
+		(start 128.778 66)
+		(end 128.778 90)
 		(stroke
 			(width 0.3)
@@
 	)
 	(gr_line
-		(start 128.778 97.7265)
-		(end 128.778 101.4095)
+		(start 129 110)
+		(end 200.5 110)
 		(stroke
-			(width 0.3)
-			(type dash)
+			(width 0.05)
+			(type default)
 		)
-		(layer "F.SilkS")
+		(layer "Edge.Cuts")
 	)
-	(gr_rect
+	(gr_line
+		(start 100.5 110)
+		(end 126 110)
+		(stroke
+			(width 0.05)
+			(type default)
+		)
+		(layer "Edge.Cuts")
+	)
+	(gr_line
+		(start 129 110)
+		(end 129 101)
+		(stroke
+			(width 0.05)
+			(type default)
+		)
+		(layer "Edge.Cuts")
+	)
+	(gr_line
+		(start 200.5 65)
+		(end 100.5 65)
+		(stroke
+			(width 0.05)
+			(type default)
+		)
+		(layer "Edge.Cuts")
+	)
+	(gr_line
+		(start 126 110)
+		(end 126 101)
+		(stroke
+			(width 0.05)
+			(type default)
+		)
+		(layer "Edge.Cuts")
+	)
+	(gr_arc
+		(start 126 101)
+		(mid 127.5 99.50085)
+		(end 129 101)
+		(stroke
+			(width 0.05)
+			(type default)
+		)
+		(layer "Edge.Cuts")
+	)
+	(gr_line
 		(start 100.5 65)
-		(end 200.5 110)
+		(end 100.5 110)
+		(stroke
+			(width 0.05)
+			(type default)
+		)
+		(layer "Edge.Cuts")
+	)
+	(gr_line
+		(start 200.5 110)
+		(end 200.5 65)
 		(stroke
 			(width 0.05)
 			(type default)
 		)
-		(fill none)
 		(layer "Edge.Cuts")
 	)
@@
 		)
 	)
-	(gr_text "ETH1ISO224 V1.1\nDefault IP : 192.168.1.21"
+	(gr_text "ETH1ISO224 V1.2\nDefault IP : 192.168.1.21"
 		(at 162.052 109.347 0)
 		(layer "F.SilkS")
@@
 	(segment
 		(start 116.713 92.386)
-		(end 118.745 94.418)
+		(end 116.713 92.7995)
 		(width 0.508)
 		(layer "B.Cu")
@@
 	)
 	(segment
-		(start 118.745 94.996)
-		(end 119.914 96.165)
+		(start 118.5 94.5865)
+		(end 118.5 95.5)
 		(width 0.508)
 		(layer "B.Cu")
@@
 	)
 	(segment
-		(start 119.914 96.165)
-		(end 120.396 96.165)
+		(start 116.713 92.7995)
+		(end 118.5 94.5865)
 		(width 0.508)
 		(layer "B.Cu")
@@
 	)
 	(segment
-		(start 118.745 94.418)
-		(end 118.745 94.996)
+		(start 119.165 96.165)
+		(end 120.396 96.165)
+		(width 0.508)
+		(layer "B.Cu")
+		(net 56)
+	)
+	(segment
+		(start 118.5 95.5)
+		(end 119.165 96.165)
 		(width 0.508)
 		(layer "B.Cu")
